File: electronics/controller/controller.kicad_pcb (KiCad board)
At the start: 2 copper layers, 20.3 x 35.6 mm, 13 parts, among them P1 CONN_01X14, P2 CONN_01X14, P3 JTAG (SWD), P4 I2C, P5 SPI, P6 UART, P7 USB_OTG, U1 LPC1114FDH28/102, U2 LP2985LV

Commit message: More work on controller
Parts:
- added C1: 10u, Capacitors_SMD:C_0805, F.Cu at (148.0, 95.2)
- added C4: 0.1u, Capacitors_SMD:C_0603, F.Cu at (148.6, 114.3)
- added SW1: ~RST~, Buttons_Switches_SMD:SW_SPST_EVQP7A, F.Cu at (144.1, 89.5)
- C2: footprint Capacitors_SMD:C_0603_HandSoldering -> Capacitors_SMD:C_0603
- C3: value 1u -> 10u; footprint Capacitors_SMD:C_0603_HandSoldering -> Capacitors_SMD:C_0805
- R1: footprint Resistors_SMD:R_0603_HandSoldering -> Resistors_SMD:R_0603
- moved C3 4.96 mm to (154.3, 95.2), turned to 90 degrees
- moved C2 2.62 mm to (151.1, 98.4), turned to 0 degrees
- moved P7 2.54 mm to (151.1, 90.2)
- moved P3 1.27 mm to (143.5, 96.5)
- moved U2 1.27 mm to (151.1, 95.2)
